Commit message: Added initial positions for uf850

File: xarm_description/urdf/lite6/lite6.ros2_control.xacro (robot description, xacro)
@@ -37,5 +37,7 @@
           <param name="max">3.14</param>
         </command_interface>
-        <state_interface name="position"/>
+        <state_interface name="position">
+          <param name="initial_value">-3.1415926536</param>
+        </state_interface>
         <state_interface name="velocity"/>
         <!-- <state_interface name="effort"/> -->
@@ -50,5 +52,7 @@
           <param name="max">3.14</param>
         </command_interface>
-        <state_interface name="position"/>
+        <state_interface name="position">
+          <param name="initial_value">-1.5707963268</param>
+        </state_interface>
         <state_interface name="velocity"/>
         <!-- <state_interface name="effort"/> -->
@@ -63,5 +67,7 @@
           <param name="max">3.14</param>
         </command_interface>
-        <state_interface name="position"/>
+        <state_interface name="position">
+          <param name="initial_value">0.0</param>
+        </state_interface>
         <state_interface name="velocity"/>
         <!-- <state_interface name="effort"/> -->
@@ -76,5 +82,7 @@
           <param name="max">3.14</param>
         </command_interface>
-        <state_interface name="position"/>
+        <state_interface name="position">
+          <param name="initial_value">-3.1415926536</param>
+        </state_interface>
         <state_interface name="velocity"/>
         <!-- <state_interface name="effort"/> -->
@@ -89,5 +97,7 @@
           <param name="max">3.14</param>
         </command_interface>
-        <state_interface name="position"/>
+        <state_interface name="position">
+          <param name="initial_value">1.5707963268</param>
+        </state_interface>
         <state_interface name="velocity"/>
         <!-- <state_interface name="effort"/> -->
@@ -102,5 +112,7 @@
           <param name="max">3.14</param>
         </command_interface>
-        <state_interface name="position"/>
+        <state_interface name="position">
+          <param name="initial_value">0</param>
+        </state_interface>
         <state_interface name="velocity"/>
         <!-- <state_interface name="effort"/> -->

File: xarm_description/urdf/uf850/uf850.ros2_control.xacro (robot description, xacro)
@@ -11,5 +11,11 @@
     joint4_lower_limit:=${-2.0*pi}  joint4_upper_limit:=${2.0*pi}
     joint5_lower_limit:=${-2.1642}  joint5_upper_limit:=${2.1642}
-    joint6_lower_limit:=${-2.0*pi}  joint6_upper_limit:=${2.0*pi}">
+    joint6_lower_limit:=${-2.0*pi}  joint6_upper_limit:=${2.0*pi} initial_positions_file:='' ">
+    <xacro:if value="${initial_positions_file != ''}">
+        <xacro:property name="initial_positions" value="${xacro.load_yaml(initial_positions_file)['initial_positions']}"/>
+    </xacro:if>
+    <xacro:unless value="${initial_positions_file != ''}">
+      <xacro:property name="initial_positions" value="false"/>
+    </xacro:unless>
     <ros2_control name="${prefix}${ros2_control_plugin}" type="system">
       <hardware>
@@ -43,5 +49,9 @@
           <param name="max">3.14</param>
         </command_interface>
-        <state_interface name="position"/>
+        <state_interface name="position">
+        <xacro:if value="${initial_positions}">
+          <param name="initial_value">${initial_positions[prefix + 'joint1']}</param>
+        </xacro:if>
+        </state_interface>
         <state_interface name="velocity"/>
         <!-- <state_interface name="effort"/> -->
@@ -56,5 +66,9 @@
           <param name="max">3.14</param>
         </command_interface>
-        <state_interface name="position"/>
+        <state_interface name="position">
+          <xacro:if value="${initial_positions}">
+          <param name="initial_value">${initial_positions[prefix + 'joint2']}</param>
+        </xacro:if>
+        </state_interface>
         <state_interface name="velocity"/>
         <!-- <state_interface name="effort"/> -->
@@ -69,5 +83,9 @@
           <param name="max">3.14</param>
         </command_interface>
-        <state_interface name="position"/>
+        <state_interface name="position">
+          <xacro:if value="${initial_positions}">
+            <param name="initial_value">${initial_positions[prefix + 'joint3']}</param>
+          </xacro:if>
+        </state_interface>
         <state_interface name="velocity"/>
         <!-- <state_interface name="effort"/> -->
@@ -82,5 +100,9 @@
           <param name="max">3.14</param>
         </command_interface>
-        <state_interface name="position"/>
+        <state_interface name="position">
+          <xacro:if value="${initial_positions}">
+          <param name="initial_value">${initial_positions[prefix + 'joint4']}</param>
+        </xacro:if>
+        </state_interface>
         <state_interface name="velocity"/>
         <!-- <state_interface name="effort"/> -->
@@ -95,5 +117,9 @@
           <param name="max">3.14</param>
         </command_interface>
-        <state_interface name="position"/>
+        <state_interface name="position">
+          <xacro:if value="${initial_positions}">
+            <param name="initial_value">${initial_positions[prefix + 'joint5']}</param>
+          </xacro:if>
+        </state_interface>
         <state_interface name="velocity"/>
         <!-- <state_interface name="effort"/> -->
@@ -108,5 +134,9 @@
           <param name="max">3.14</param>
         </command_interface>
-        <state_interface name="position"/>
+        <state_interface name="position">
+          <xacro:if value="${initial_positions}">
+            <param name="initial_value">${initial_positions[prefix + 'joint6']}</param>
+          </xacro:if>
+        </state_interface>
         <state_interface name="velocity"/>
         <!-- <state_interface name="effort"/> -->

File: xarm_description/urdf/uf850/uf850.urdf.xacro (robot description, xacro)
@@ -8,6 +8,5 @@
     joint5_lower_limit:=${-2.1642}  joint5_upper_limit:=${2.1642}
     joint6_lower_limit:=${-2.0*pi}  joint6_upper_limit:=${2.0*pi}
-    model1300:=false
-    inertial_params_filename:='' kinematics_params_filename:='' "
+    model1300:=false inertial_params_filename:='' kinematics_params_filename:='' "
     >
     <!-- load params and define property -->

File: xarm_description/urdf/uf850/uf850_robot_macro.xacro (robot description, xacro)
@@ -15,5 +15,5 @@
     inertial_params_filename:=''
     kinematics_params_filename:=''
-    hard_interface:='PositionJointInterface' "
+    hard_interface:='PositionJointInterface' initial_positions_file:='' "
     >
     <!-- include uf850 relative macros: -->
@@ -37,5 +37,5 @@
           joint4_lower_limit="${-pi*0.99}" joint4_upper_limit="${pi*0.99}"
           joint5_lower_limit="${-2.1642}" joint5_upper_limit="${2.1642}"
-          joint6_lower_limit="${-pi*0.99}" joint6_upper_limit="${pi*0.99}"/>
+          joint6_lower_limit="${-pi*0.99}" joint6_upper_limit="${pi*0.99}" initial_positions_file="${initial_positions_file}"/>
       </xacro:if>
       <xacro:uf850_urdf prefix="${prefix}"
@@ -56,5 +56,5 @@
           hw_ns="${hw_ns}" add_gripper="${add_gripper}"
           robot_ip="${robot_ip}" report_type="${report_type}"
-          baud_checkset="${baud_checkset}" default_gripper_baud="${default_gripper_baud}" />
+          baud_checkset="${baud_checkset}" default_gripper_baud="${default_gripper_baud}" initial_positions_file="${initial_positions_file}" />
       </xacro:if>
       <xacro:uf850_urdf prefix="${prefix}" model1300="${model1300}"

File: xarm_description/urdf/xarm_device.urdf.xacro (robot description, xacro)
@@ -38,4 +38,5 @@
   <xacro:arg name="mesh_suffix" default="stl"/>
   <xacro:arg name="kinematics_suffix" default=""/>
+  <xacro:arg name="initial_positions_file" default=""/>
   <!-- load xarm device -->
   <xacro:include filename="$(find xarm_description)/urdf/xarm_device_macro.xacro" />
@@ -57,4 +58,4 @@
     baud_checkset="$(arg baud_checkset)" default_gripper_baud="$(arg default_gripper_baud)"
     model1300="$(arg model1300)" attach_to="$(arg attach_to)" attach_xyz="$(arg attach_xyz)" attach_rpy="$(arg attach_rpy)"
-    robot_sn="$(arg robot_sn)" use_gazebo_camera="$(arg use_gazebo_camera)" mesh_suffix="$(arg mesh_suffix)" kinematics_suffix="$(arg kinematics_suffix)" />
+    robot_sn="$(arg robot_sn)" use_gazebo_camera="$(arg use_gazebo_camera)" mesh_suffix="$(arg mesh_suffix)" kinematics_suffix="$(arg kinematics_suffix)" initial_positions_file="$(arg initial_positions_file)" />
 </robot>

File: xarm_description/urdf/xarm_device_macro.xacro (robot description, xacro)
@@ -39,5 +39,5 @@
     model1300:=false
     robot_sn:=''
-    mesh_suffix:='stl'
+    mesh_suffix:='stl' initial_positions_file:=''
     kinematics_suffix:=''
     "
@@ -109,5 +109,7 @@
         inertial_params_filename="${inertial_params_filename}"
         kinematics_params_filename="${kinematics_params_filename}"
-        hard_interface="${hard_interface}" />
+        hard_interface="${hard_interface}"
+        initial_positions_file="${initial_positions_file}"
+       />
     </xacro:if>
     <xacro:if value="${dof == 6}">
@@ -126,5 +128,6 @@
           inertial_params_filename="${inertial_params_filename}"
           kinematics_params_filename="${kinematics_params_filename}"
-          hard_interface="${hard_interface}" />
+          hard_interface="${hard_interface}"
+          initial_positions_file="${initial_positions_file}" />
       </xacro:if>
       <xacro:if value="${robot_type == 'lite'}">
@@ -141,5 +144,7 @@
           inertial_params_filename="${inertial_params_filename}"
           kinematics_params_filename="${kinematics_params_filename}"
-          hard_interface="${hard_interface}" />
+          hard_interface="${hard_interface}"
+          initial_positions_file="${initial_positions_file}"
+         />
       </xacro:if>
       <xacro:unless value="${robot_type == 'lite' or robot_type == 'uf850'}">
@@ -157,5 +162,7 @@
           inertial_params_filename="${inertial_params_filename}"
           kinematics_params_filename="${kinematics_params_filename}"
-          hard_interface="${hard_interface}" />
+          hard_interface="${hard_interface}"
+          initial_positions_file="${initial_positions_file}"
+         />
       </xacro:unless>
     </xacro:if>
@@ -174,5 +181,7 @@
         inertial_params_filename="${inertial_params_filename}"
         kinematics_params_filename="${kinematics_params_filename}"
-        hard_interface="${hard_interface}" />
+        hard_interface="${hard_interface}"
+        initial_positions_file="${initial_positions_file}"
+       />
     </xacro:unless>
     <xacro:if value="${add_realsense_d435i}">
