Commit message: removed world joint

File: xarm_moveit_config/srdf/_lite6_macro.srdf.xacro (robot description, xacro)
@@ -9,8 +9,7 @@
   <!-- CHAINS: When a chain is specified, all the links along the chain (including endpoints) are included in the group. Additionally, all the joints that are parents to included links are also included. This means that joints along the chain and the parent joint of the base link are included in the group -->
   <!-- SUBGROUPS: Groups can also be formed by referencing to already defined group names -->
-  <xacro:macro name="lite6_macro_srdf" params="prefix=''
-    add_gripper='false' add_vacuum_gripper='false' add_other_geometry='false' ">
+  <xacro:macro name="lite6_macro_srdf" params="prefix='' add_gripper='false' add_vacuum_gripper='false' add_other_geometry='false' ">
     <group name="${prefix}lite6">
-      <joint name="${prefix}world_joint" />
+      <!-- <joint name="${prefix}world_joint" /> -->
       <joint name="${prefix}joint1" />
       <joint name="${prefix}joint2" />
